Commit message: init change IP`s

File: src/ur_dual_control/urdf/ur_dual_controlled.urdf.xacro (robot description, xacro)
@@ -1,35 +1,34 @@
 <?xml version="1.0"?>
 <robot name="ur_dual" xmlns:xacro="http://ros.org/wiki/xacro">
-  <!-- Include the dual-arm macro and ROS2 control definitions -->
+  <!-- Incluir las definiciones necesarias -->
   <xacro:include filename="$(find ur_dual_description)/urdf/ur_dual_macro.xacro"/>
   <xacro:include filename="$(find ur_description)/urdf/ur.ros2_control.xacro"/>
-  <!-- Define the arguments for parametrization using I and D naming -->
+  <!-- Definir argumentos -->
   <xacro:arg name="ur_type_I" default="ur5e"/>
   <xacro:arg name="ur_type_D" default="ur5e"/>
-  <xacro:arg name="ur_type" default="ur5e"/>
   <xacro:arg name="robot_ip_I" default="10.113.36.96"/>
   <xacro:arg name="robot_ip_D" default="10.113.36.97"/>
-  <xacro:arg name="joint_limits_parameters_file_I" default="$(find ur_description)/config/$(arg ur_type_I)/joint_limits.yaml"/>
-  <xacro:arg name="joint_limits_parameters_file_D" default="$(find ur_description)/config/$(arg ur_type_D)/joint_limits.yaml"/>
-  <xacro:arg name="kinematics_parameters_file_I" default="$(find ur_description)/config/$(arg ur_type_I)/default_kinematics.yaml"/>
-  <xacro:arg name="kinematics_parameters_file_D" default="$(find ur_description)/config/$(arg ur_type_D)/default_kinematics.yaml"/>
-  <xacro:arg name="physical_parameters_file_I" default="$(find ur_description)/config/$(arg ur_type_I)/physical_parameters.yaml"/>
-  <xacro:arg name="physical_parameters_file_D" default="$(find ur_description)/config/$(arg ur_type_D)/physical_parameters.yaml"/>
-  <xacro:arg name="visual_parameters_file_I" default="$(find ur_description)/config/$(arg ur_type_I)/visual_parameters.yaml"/>
-  <xacro:arg name="visual_parameters_file_D" default="$(find ur_description)/config/$(arg ur_type_D)/visual_parameters.yaml"/>
-  <xacro:arg name="headless_mode" default="false"/>
-  <xacro:arg name="use_mock_hardware" default="false"/>
-  <xacro:arg name="mock_sensor_commands" default="false"/>
-  <xacro:arg name="ur_script_filename" default="$(find ur_client_library)/resources/external_control.urscript"/>
-  <xacro:arg name="ur_output_recipe_filename" default="$(find ur_robot_driver)/resources/rtde_output_recipe.txt"/>
-  <xacro:arg name="ur_input_recipe_filename" default="$(find ur_robot_driver)/resources/rtde_input_recipe.txt"/>
+  <xacro:arg name="joint_limits_parameters_file_I"
+             default="$(find ur_description)/config/$(arg ur_type_I)/joint_limits.yaml"/>
+  <xacro:arg name="joint_limits_parameters_file_D"
+             default="$(find ur_description)/config/$(arg ur_type_D)/joint_limits.yaml"/>
+  <xacro:arg name="kinematics_parameters_file_I"
+             default="$(find ur_description)/config/$(arg ur_type_I)/default_kinematics.yaml"/>
+  <xacro:arg name="kinematics_parameters_file_D"
+             default="$(find ur_description)/config/$(arg ur_type_D)/default_kinematics.yaml"/>
+  <xacro:arg name="physical_parameters_file_I"
+             default="$(find ur_description)/config/$(arg ur_type_I)/physical_parameters.yaml"/>
+  <xacro:arg name="physical_parameters_file_D"
+             default="$(find ur_description)/config/$(arg ur_type_D)/physical_parameters.yaml"/>
+  <xacro:arg name="visual_parameters_file_I"
+             default="$(find ur_description)/config/$(arg ur_type_I)/visual_parameters.yaml"/>
+  <xacro:arg name="visual_parameters_file_D"
+             default="$(find ur_description)/config/$(arg ur_type_D)/visual_parameters.yaml"/>
   <xacro:arg name="namespace" default="ur_dual"/>
-  <xacro:arg name="hash_kinematics" default="false"/>
-  <!-- Define world link -->
-  <link name="world"/>
-  <!-- Instantiate the dual-arm robot using the I and D parameters -->
+  <!-- Instanciar la macro con los dos brazos -->
   <xacro:ur_dual
     parent="world"
-    ur_type="$(arg ur_type_D)"
+    ur_type_I="$(arg ur_type_I)"
+    ur_type_D="$(arg ur_type_D)"
     joint_limits_parameters_file_I="$(arg joint_limits_parameters_file_I)"
     joint_limits_parameters_file_D="$(arg joint_limits_parameters_file_D)"
@@ -40,29 +39,6 @@
     visual_parameters_file_I="$(arg visual_parameters_file_I)"
     visual_parameters_file_D="$(arg visual_parameters_file_D)"
-    namespace="$(arg namespace)"
-  >
+    namespace="$(arg namespace)">
     <origin xyz="0 0 0" rpy="0 0 0"/>
   </xacro:ur_dual>
-  <!-- ROS2 Control configuration for the first UR5e (arm I) -->
-  <xacro:ur_ros2_control
-    name="ur_dual_I"
-    tf_prefix="ur_dual_I_"
-    robot_ip="$(arg robot_ip_I)"
-    script_filename="$(arg ur_script_filename)"
-    output_recipe_filename="$(arg ur_output_recipe_filename)"
-    input_recipe_filename="$(arg ur_input_recipe_filename)"
-    headless_mode="$(arg headless_mode)"
-    hash_kinematics="$(arg hash_kinematics)"
-  />
-  <!-- ROS2 Control configuration for the second UR5e (arm D) -->
-  <xacro:ur_ros2_control
-    name="ur_dual_D"
-    tf_prefix="ur_dual_D_"
-    robot_ip="$(arg robot_ip_D)"
-    script_filename="$(arg ur_script_filename)"
-    output_recipe_filename="$(arg ur_output_recipe_filename)"
-    input_recipe_filename="$(arg ur_input_recipe_filename)"
-    headless_mode="$(arg headless_mode)"
-    hash_kinematics="$(arg hash_kinematics)"
-  />
 </robot>

File: src/ur_dual_description/urdf/ur_dual.urdf.xacro (robot description, xacro)
@@ -1,22 +1,33 @@
 <?xml version="1.0"?>
 <robot name="ur_dual" xmlns:xacro="http://ros.org/wiki/xacro">
+  <!-- Definir el link "world" al inicio para que esté disponible para todos los joints -->
+  <link name="world"/>
   <xacro:include filename="$(find ur_dual_description)/urdf/ur_dual_macro.xacro"/>
-  <xacro:arg name="ur_type" default="ur5e"/>
-  <xacro:arg name="joint_limits_parameters_file" default="$(find ur_description)/config/$(arg ur_type)/joint_limits.yaml"/>
-  <xacro:arg name="kinematics_parameters_file" default="$(find ur_description)/config/$(arg ur_type)/default_kinematics.yaml"/>
-  <xacro:arg name="physical_parameters_file" default="$(find ur_description)/config/$(arg ur_type)/physical_parameters.yaml"/>
-  <xacro:arg name="visual_parameters_file" default="$(find ur_description)/config/$(arg ur_type)/visual_parameters.yaml"/>
+  <!-- Se definen argumentos separados para cada brazo -->
+  <xacro:arg name="ur_type_I" default="ur5e"/>
+  <xacro:arg name="ur_type_D" default="ur5e"/>
+  <xacro:arg name="joint_limits_parameters_file_I" default="$(find ur_description)/config/$(arg ur_type_I)/joint_limits.yaml"/>
+  <xacro:arg name="kinematics_parameters_file_I" default="$(find ur_description)/config/$(arg ur_type_I)/default_kinematics.yaml"/>
+  <xacro:arg name="physical_parameters_file_I" default="$(find ur_description)/config/$(arg ur_type_I)/physical_parameters.yaml"/>
+  <xacro:arg name="visual_parameters_file_I" default="$(find ur_description)/config/$(arg ur_type_I)/visual_parameters.yaml"/>
+  <xacro:arg name="joint_limits_parameters_file_D" default="$(find ur_description)/config/$(arg ur_type_D)/joint_limits.yaml"/>
+  <xacro:arg name="kinematics_parameters_file_D" default="$(find ur_description)/config/$(arg ur_type_D)/default_kinematics.yaml"/>
+  <xacro:arg name="physical_parameters_file_D" default="$(find ur_description)/config/$(arg ur_type_D)/physical_parameters.yaml"/>
+  <xacro:arg name="visual_parameters_file_D" default="$(find ur_description)/config/$(arg ur_type_D)/visual_parameters.yaml"/>
   <xacro:arg name="namespace" default="ur_dual"/>
-  <link name="world"/>
-  <!--This will create the scene where the robot is located in-->
+  <!-- Instanciar la macro, la cual ahora recibe los parámetros específicos para cada brazo -->
   <xacro:ur_dual
     parent="world"
-    ur_type="$(arg ur_type)"
-    joint_limits_parameters_file="$(arg joint_limits_parameters_file)"
-    kinematics_parameters_file="$(arg kinematics_parameters_file)"
-    physical_parameters_file="$(arg physical_parameters_file)"
-    visual_parameters_file="$(arg visual_parameters_file)"
-    namespace="$(arg namespace)"
-    >
+    ur_type_I="$(arg ur_type_I)"
+    ur_type_D="$(arg ur_type_D)"
+    joint_limits_parameters_file_I="$(arg joint_limits_parameters_file_I)"
+    joint_limits_parameters_file_D="$(arg joint_limits_parameters_file_D)"
+    kinematics_parameters_file_I="$(arg kinematics_parameters_file_I)"
+    kinematics_parameters_file_D="$(arg kinematics_parameters_file_D)"
+    physical_parameters_file_I="$(arg physical_parameters_file_I)"
+    physical_parameters_file_D="$(arg physical_parameters_file_D)"
+    visual_parameters_file_I="$(arg visual_parameters_file_I)"
+    visual_parameters_file_D="$(arg visual_parameters_file_D)"
+    namespace="$(arg namespace)">
       <origin xyz="0 0 1" rpy="0 0 0" />
   </xacro:ur_dual>

File: src/ur_dual_description/urdf/ur_dual_macro.xacro (robot description, xacro)
@@ -2,14 +2,21 @@
 <robot xmlns:xacro="http://ros.org/wiki/xacro">
   <xacro:include filename="$(find ur_description)/urdf/ur_macro.xacro"/>
+  <!-- Macro para definir los dos brazos del UR -->
   <xacro:macro name="ur_dual" params="
     parent
     *origin
-    ur_type
-    joint_limits_parameters_file
-    kinematics_parameters_file
-    physical_parameters_file
-    visual_parameters_file
+    ur_type_I
+    ur_type_D
+    joint_limits_parameters_file_I
+    joint_limits_parameters_file_D
+    kinematics_parameters_file_I
+    kinematics_parameters_file_D
+    physical_parameters_file_I
+    physical_parameters_file_D
+    visual_parameters_file_I
+    visual_parameters_file_D
     namespace
     ">
+    <!-- Base para el brazo izquierdo (I) -->
     <link name="robot_mount_I"/>
     <joint name="base_to_robot_mount_I" type="fixed">
@@ -18,4 +25,5 @@
       <origin xyz="0.46 0 0" rpy="0 0 0" />
     </joint>
+    <!-- Base para el brazo derecho (D) -->
     <link name="robot_mount_D"/>
     <joint name="base_to_robot_mount_D" type="fixed">
@@ -24,24 +32,25 @@
       <origin xyz="-0.46 0 0" rpy="0 0 0" />
     </joint>
-    <!--This will create the specific robot-->
+    <!-- Definición del brazo izquierdo (I) -->
     <xacro:ur_robot
-      name="${ur_type}_I"
+      name="${ur_type_I}_I"
       tf_prefix="${namespace}_I_"
       parent="robot_mount_I"
-      joint_limits_parameters_file="${joint_limits_parameters_file}"
-      kinematics_parameters_file="${kinematics_parameters_file}"
-      physical_parameters_file="${physical_parameters_file}"
-      visual_parameters_file="${visual_parameters_file}"
+      joint_limits_parameters_file="${joint_limits_parameters_file_I}"
+      kinematics_parameters_file="${kinematics_parameters_file_I}"
+      physical_parameters_file="${physical_parameters_file_I}"
+      visual_parameters_file="${visual_parameters_file_I}"
     >
       <origin xyz="0 0 0" rpy="0 0 0" />
     </xacro:ur_robot>
+    <!-- Definición del brazo derecho (D) -->
     <xacro:ur_robot
-      name="${ur_type}_D"
+      name="${ur_type_D}_D"
       tf_prefix="${namespace}_D_"
       parent="robot_mount_D"
-      joint_limits_parameters_file="${joint_limits_parameters_file}"
-      kinematics_parameters_file="${kinematics_parameters_file}"
-      physical_parameters_file="${physical_parameters_file}"
-      visual_parameters_file="${visual_parameters_file}"
+      joint_limits_parameters_file="${joint_limits_parameters_file_D}"
+      kinematics_parameters_file="${kinematics_parameters_file_D}"
+      physical_parameters_file="${physical_parameters_file_D}"
+      visual_parameters_file="${visual_parameters_file_D}"
     >
       <origin xyz="0 0 0" rpy="0 0 0" />
@@ -52,9 +61,8 @@
         <geometry>
           <box size="2.0 2.0 0.01"/>
-          <!-- Dimensiones del plano 20m x 20m x 0.01m -->
         </geometry>
-        <origin xyz="0 0 -0.005" rpy="0 0 0"/> <!-- Colocado en z=0 -->
+        <origin xyz="0 0 -0.005" rpy="0 0 0"/>
         <material name="floor_material">
-          <color rgba="0.8 0.8 0.8 1.0"/> <!-- Color gris claro -->
+          <color rgba="0.8 0.8 0.8 1.0"/>
         </material>
       </visual>
@@ -66,5 +74,5 @@
       </collision>
       <inertial>
-        <mass value="1.0"/> <!-- Masa arbitraria -->
+        <mass value="1.0"/>
         <origin xyz="0 0 -0.005" rpy="0 0 0"/>
         <inertia ixx="0.01" iyy="0.01" izz="0.01" ixy="0.0" ixz="0.0" iyz="0.0"/>

Commit message: Joints states working

File: src/ur_dual_control/urdf/ur_dual_controlled.urdf.xacro (robot description, xacro)
@@ -4,26 +4,46 @@
   <xacro:include filename="$(find ur_dual_description)/urdf/ur_dual_macro.xacro"/>
   <xacro:include filename="$(find ur_description)/urdf/ur.ros2_control.xacro"/>
+  <xacro:include filename="$(find ur_description)/urdf/inc/ur_common.xacro"/>
   <!-- Definir argumentos -->
-  <xacro:arg name="ur_type_I" default="ur5e"/>
-  <xacro:arg name="ur_type_D" default="ur5e"/>
-  <xacro:arg name="robot_ip_I" default="10.113.36.96"/>
-  <xacro:arg name="robot_ip_D" default="10.113.36.97"/>
-  <xacro:arg name="joint_limits_parameters_file_I"
-             default="$(find ur_description)/config/$(arg ur_type_I)/joint_limits.yaml"/>
-  <xacro:arg name="joint_limits_parameters_file_D"
-             default="$(find ur_description)/config/$(arg ur_type_D)/joint_limits.yaml"/>
-  <xacro:arg name="kinematics_parameters_file_I"
-             default="$(find ur_description)/config/$(arg ur_type_I)/default_kinematics.yaml"/>
-  <xacro:arg name="kinematics_parameters_file_D"
-             default="$(find ur_description)/config/$(arg ur_type_D)/default_kinematics.yaml"/>
-  <xacro:arg name="physical_parameters_file_I"
-             default="$(find ur_description)/config/$(arg ur_type_I)/physical_parameters.yaml"/>
-  <xacro:arg name="physical_parameters_file_D"
-             default="$(find ur_description)/config/$(arg ur_type_D)/physical_parameters.yaml"/>
-  <xacro:arg name="visual_parameters_file_I"
-             default="$(find ur_description)/config/$(arg ur_type_I)/visual_parameters.yaml"/>
-  <xacro:arg name="visual_parameters_file_D"
-             default="$(find ur_description)/config/$(arg ur_type_D)/visual_parameters.yaml"/>
   <xacro:arg name="namespace" default="ur_dual"/>
+  <xacro:arg name="sim_gazebo" default="false"/>
+  <xacro:arg name="sim_ignition" default="false"/>
+    <!--We need to specify the arguments used for parametrizing our description-->
+  <xacro:arg name="ur_type_I" default="ur5e" />
+  <xacro:arg name="joint_limits_parameters_file_I" default="$(find ur_description)/config/$(arg ur_type_I)/joint_limits.yaml" />
+  <xacro:arg name="kinematics_parameters_file_I" default="$(find ur_description)/config/$(arg ur_type_I)/default_kinematics.yaml" />
+  <xacro:arg name="physical_parameters_file_I" default="$(find ur_description)/config/$(arg ur_type_I)/physical_parameters.yaml" />
+  <xacro:arg name="visual_parameters_file_I" default="$(find ur_description)/config/$(arg ur_type_I)/visual_parameters.yaml" />
+  <xacro:arg name="ur_type_D" default="ur5e" />
+  <xacro:arg name="joint_limits_parameters_file_D" default="$(find ur_description)/config/$(arg ur_type_D)/joint_limits.yaml" />
+  <xacro:arg name="kinematics_parameters_file_D" default="$(find ur_description)/config/$(arg ur_type_D)/default_kinematics.yaml" />
+  <xacro:arg name="physical_parameters_file_D" default="$(find ur_description)/config/$(arg ur_type_D)/physical_parameters.yaml" />
+  <xacro:arg name="visual_parameters_file_D" default="$(find ur_description)/config/$(arg ur_type_D)/visual_parameters.yaml" />
+  <xacro:arg name="use_mock_hardware_I" default="false" />
+  <xacro:arg name="mock_sensor_commands_I" default="false" />
+  <xacro:arg name="robot_ip_I" default="10.113.36.100" />
+  <xacro:arg name="reverse_port_I" default="50006" />
+  <xacro:arg name="script_sender_port_I" default="50007" />
+  <xacro:arg name="script_command_port_I" default="50010" />
+  <xacro:arg name="trajectory_port_I" default="50009" />
+  <xacro:arg name="use_mock_hardware_D" default="false" />
+  <xacro:arg name="mock_sensor_commands_D" default="false" />
+  <xacro:arg name="robot_ip_D" default="10.113.36.247" />
+  <xacro:arg name="reverse_port_D" default="50001" />
+  <xacro:arg name="script_sender_port_D" default="50002" />
+  <xacro:arg name="script_command_port_D" default="50004" />
+  <xacro:arg name="trajectory_port_D" default="50003" />
+  <xacro:arg name="headless_mode" default="false" />
+  <xacro:arg name="ur_script_filename" default="$(find ur_client_library)/resources/external_control.urscript" />
+  <xacro:arg name="ur_output_recipe_filename" default="$(find ur_robot_driver)/resources/rtde_output_recipe.txt" />
+  <xacro:arg name="ur_input_recipe_filename" default="$(find ur_robot_driver)/resources/rtde_input_recipe.txt" />
+   <!-- Load configuration data from the provided .yaml files -->
+  <xacro:read_model_data
+     joint_limits_parameters_file="$(arg joint_limits_parameters_file_I)"
+     kinematics_parameters_file="$(arg kinematics_parameters_file_I)"
+     physical_parameters_file="$(arg physical_parameters_file_I)"
+     visual_parameters_file="$(arg visual_parameters_file_I)"
+     force_abs_paths="$(arg sim_gazebo)"/>
+  <link name="world"/>
   <!-- Instanciar la macro con los dos brazos -->
   <xacro:ur_dual
@@ -39,6 +59,38 @@
     visual_parameters_file_I="$(arg visual_parameters_file_I)"
     visual_parameters_file_D="$(arg visual_parameters_file_D)"
-    namespace="$(arg namespace)">
+    >
     <origin xyz="0 0 0" rpy="0 0 0"/>
   </xacro:ur_dual>
+   <xacro:ur_ros2_control
+    name="ur_dual_I"
+    tf_prefix="ur_dual_I_"
+    robot_ip="$(arg robot_ip_I)"
+    hash_kinematics="${kinematics_hash}"
+    script_filename="$(arg ur_script_filename)"
+    output_recipe_filename="$(arg ur_output_recipe_filename)"
+    input_recipe_filename="$(arg ur_input_recipe_filename)"
+    use_fake_hardware="$(arg use_mock_hardware_I)"
+    fake_sensor_commands="$(arg mock_sensor_commands_I)"
+    headless_mode="$(arg headless_mode)"
+    reverse_port="$(arg reverse_port_I)"
+    script_sender_port="$(arg script_sender_port_I)"
+    script_command_port="$(arg script_command_port_I)"
+    trajectory_port="$(arg trajectory_port_I)"
+  />
+  <xacro:ur_ros2_control
+    name="ur_dual_D"
+    tf_prefix="ur_dual_D_"
+    robot_ip="$(arg robot_ip_D)"
+    hash_kinematics="${kinematics_hash}"
+    script_filename="$(arg ur_script_filename)"
+    output_recipe_filename="$(arg ur_output_recipe_filename)"
+    input_recipe_filename="$(arg ur_input_recipe_filename)"
+    use_fake_hardware="$(arg use_mock_hardware_D)"
+    fake_sensor_commands="$(arg mock_sensor_commands_D)"
+    headless_mode="$(arg headless_mode)"
+    reverse_port="$(arg reverse_port_D)"
+    script_sender_port="$(arg script_sender_port_D)"
+    script_command_port="$(arg script_command_port_D)"
+    trajectory_port="$(arg trajectory_port_D)"
+  />
 </robot>

File: src/ur_dual_description/urdf/ur_dual_macro.xacro (robot description, xacro)
@@ -16,10 +16,9 @@
     visual_parameters_file_I
     visual_parameters_file_D
-    namespace
     ">
     <!-- Base para el brazo izquierdo (I) -->
     <link name="robot_mount_I"/>
     <joint name="base_to_robot_mount_I" type="fixed">
-      <parent link="world"/>
+      <parent link="floor"/>
       <child link="robot_mount_I"/>
       <origin xyz="0.46 0 0" rpy="0 0 0" />
@@ -28,12 +27,12 @@
     <link name="robot_mount_D"/>
     <joint name="base_to_robot_mount_D" type="fixed">
-      <parent link="world"/>
+      <parent link="floor"/>
       <child link="robot_mount_D"/>
       <origin xyz="-0.46 0 0" rpy="0 0 0" />
     </joint>
     <!-- Definición del brazo izquierdo (I) -->
-    <xacro:ur_robot
-      name="${ur_type_I}_I"
-      tf_prefix="${namespace}_I_"
+    <!-- <xacro:ur_robot
+      name="ur_dual_I"
+      tf_prefix="ur_dual_I_"
       parent="robot_mount_I"
       joint_limits_parameters_file="${joint_limits_parameters_file_I}"
@@ -43,9 +42,9 @@
     >
       <origin xyz="0 0 0" rpy="0 0 0" />
-    </xacro:ur_robot>
+    </xacro:ur_robot> -->
     <!-- Definición del brazo derecho (D) -->
-    <xacro:ur_robot
-      name="${ur_type_D}_D"
-      tf_prefix="${namespace}_D_"
+    <!-- <xacro:ur_robot
+      name="ur_dual_D"
+      tf_prefix="ur_dual_D_"
       parent="robot_mount_D"
       joint_limits_parameters_file="${joint_limits_parameters_file_D}"
@@ -55,5 +54,5 @@
     >
       <origin xyz="0 0 0" rpy="0 0 0" />
-    </xacro:ur_robot>
+    </xacro:ur_robot> -->
     <!-- Agregar un plano al entorno -->
     <link name="floor">
