Commit message: feat: add qbhand2m.urdf.xacro inclusion and wrist joint for SoftHand integration

File: src/ur_dual_description/urdf/ur_dual_macro.xacro (robot description, xacro)
@@ -2,4 +2,5 @@
 <robot xmlns:xacro="http://ros.org/wiki/xacro">
   <xacro:include filename="$(find ur_description)/urdf/ur_macro.xacro"/>
+  <xacro:include filename="$(find qb_hand_description)/urdf/qbhand2m.urdf.xacro"/>
   <!-- Macro para definir los dos brazos del UR -->
   <xacro:macro name="ur_dual" params="
@@ -44,4 +45,10 @@
       <origin xyz="0 0 0" rpy="0 0 0" />
     </xacro:ur_robot>
+    <!-- Conectar la SoftHand al UR5e -->
+    <joint name="wrist_3_to_hand_mount" type="fixed">
+      <parent link="ur_dual_I_tool0"/>
+      <child link="root_link"/> <!-- Enlace base de la SoftHand -->
+      <origin xyz="0 0 0" rpy="0 0 0"/> <!-- Ajusta el offset según sea necesario -->
+    </joint>
     <!-- Definición del brazo derecho (D) -->
     <xacro:ur_robot

Commit message: feat: update package.xml and launch files for qbhand2m integration

File: src/ur_dual_description/urdf/ur_dual_macro.xacro (robot description, xacro)
@@ -2,5 +2,4 @@
 <robot xmlns:xacro="http://ros.org/wiki/xacro">
   <xacro:include filename="$(find ur_description)/urdf/ur_macro.xacro"/>
-  <xacro:include filename="$(find qb_hand_description)/urdf/qbhand2m.urdf.xacro"/>
   <!-- Macro para definir los dos brazos del UR -->
   <xacro:macro name="ur_dual" params="
@@ -45,10 +44,4 @@
       <origin xyz="0 0 0" rpy="0 0 0" />
     </xacro:ur_robot>
-    <!-- Conectar la SoftHand al UR5e -->
-    <joint name="wrist_3_to_hand_mount" type="fixed">
-      <parent link="ur_dual_I_tool0"/>
-      <child link="root_link"/> <!-- Enlace base de la SoftHand -->
-      <origin xyz="0 0 0" rpy="0 0 0"/> <!-- Ajusta el offset según sea necesario -->
-    </joint>
     <!-- Definición del brazo derecho (D) -->
     <xacro:ur_robot

Commit message: feat: add debug logging and update timeout in launch files; include qbhand in URDF

File: src/ur_dual_description/urdf/ur_dual_macro.xacro (robot description, xacro)
@@ -2,4 +2,11 @@
 <robot xmlns:xacro="http://ros.org/wiki/xacro">
   <xacro:include filename="$(find ur_description)/urdf/ur_macro.xacro"/>
+  <xacro:include filename="$(find qb_hand_description)/urdf/qbhand.utils.xacro"/>
+	<xacro:arg name="namespace" default="qbhand2m1"/>
+	<xacro:arg name="generate_control_tag" default="false"/>
+	<link name="root_link"/>
+	<xacro:build_hand_2m_from_yaml configuration="qbhand_right" namespace="$(arg namespace)" parent="root" generate_control_tag="$(arg generate_control_tag)">
+		<origin xyz="0 0 0" rpy="0 0 0"/>
+	</xacro:build_hand_2m_from_yaml>
   <!-- Macro para definir los dos brazos del UR -->
   <xacro:macro name="ur_dual" params="
@@ -44,4 +51,10 @@
       <origin xyz="0 0 0" rpy="0 0 0" />
     </xacro:ur_robot>
+     <!-- Conectar la SoftHand al UR5e -->
+    <joint name="wrist_3_to_hand_mount" type="fixed">
+      <parent link="ur_dual_I_tool0"/>
+      <child link="root_link"/> <!-- Enlace base de la SoftHand -->
+      <origin xyz="0 0 0" rpy="0 0 0"/> <!-- Ajusta el offset según sea necesario -->
+    </joint>
     <!-- Definición del brazo derecho (D) -->
     <xacro:ur_robot

Commit message: feat: add OnRobot 2FG7 gripper package with URDF, launch files, and Gazebo integration

File: src/ur_dual_description/urdf/ur_dual_macro.xacro (robot description, xacro)
@@ -3,4 +3,5 @@
   <xacro:include filename="$(find ur_description)/urdf/ur_macro.xacro"/>
   <xacro:include filename="$(find qb_hand_description)/urdf/qbhand.utils.xacro"/>
+  <xacro:include filename="$(find onrobot_gripper)/urdf/onrobot_2fg7_upload.xacro"/>
 	<xacro:arg name="namespace" default="qbhand2m1"/>
 	<xacro:arg name="generate_control_tag" default="false"/>
@@ -57,4 +58,9 @@
       <origin xyz="0 0 0" rpy="0 0 0"/> <!-- Ajusta el offset según sea necesario -->
     </joint>
+    <joint name="world_joint" type="fixed">
+      <parent link="ur_dual_D_tool0" />
+      <child link = "base_link" />
+      <origin xyz="0.0 0.0 0.0" rpy="0.0 0.0 0.0" />
+    </joint>
     <!-- Definición del brazo derecho (D) -->
     <xacro:ur_robot
